File: OLED_Module/KiCad/neutrino_display.kicad_sch (KiCad schematic)
At the start: 5 parts, among them J2 OLED_Headers, SW1 EC11_Switch, SW2 Kill Switch

Commit message: Fixed PCBs, updated firmware, added PrusaSlicer settings, updated README.md, updated BOM. Awesome :)
Connections:
- net +5V: now also J2.2 (Pin_2); no longer J2.1 (Pin_1)
- net GND: now also J2.1 (Pin_1); no longer J2.2 (Pin_2)
Changed lines of the file:
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@@
     (stroke (width 0) (type default))
   )
-  (wire (pts (xy 86.36 72.39) (xy 86.36 73.66))
+  (wire (pts (xy 86.36 72.39) (xy 86.36 78.74))
     (stroke (width 0) (type default))
   )
@@
     (stroke (width 0) (type default))
   )
+  (wire (pts (xy 86.36 78.74) (xy 72.39 78.74))
+    (stroke (width 0) (type default))
+  )
   (wire (pts (xy 64.77 78.74) (xy 36.83 78.74))
     (stroke (width 0) (type default))
@@
     (stroke (width 0) (type default))
   )
-  (wire (pts (xy 80.01 73.66) (xy 86.36 73.66))
-    (stroke (width 0) (type default))
-  )
   (wire (pts (xy 36.83 68.58) (xy 49.53 68.58))
     (stroke (width 0) (type default))
   )
-  (wire (pts (xy 80.01 72.39) (xy 83.82 72.39))
+  (wire (pts (xy 72.39 72.39) (xy 83.82 72.39))
     (stroke (width 0) (type default))
   )
@@
     )
   )
-  (symbol (lib_id "power:+5V") (at 80.01 72.39 0) (unit 1)
-    (in_bom yes) (on_board yes) (dnp no) (fields_autoplaced)
-    (property "Reference" "#PWR03" (at 80.01 76.2 0)
-      (effects (font (size 1.27 1.27)) hide)
-    )
-    (property "Value" "+5V" (at 80.01 68.58 0)
-      (effects (font (size 1.27 1.27)))
-    )
-    (property "Footprint" "" (at 80.01 72.39 0)
-      (effects (font (size 1.27 1.27)) hide)
-    )
-    (property "Datasheet" "" (at 80.01 72.39 0)
+  (symbol (lib_id "power:GND") (at 72.39 72.39 0) (unit 1)
+    (in_bom yes) (on_board yes) (dnp no)
+    (property "Reference" "#PWR03" (at 72.39 78.74 0)
+      (effects (font (size 1.27 1.27)) hide)
+    )
+    (property "Value" "GND" (at 72.39 71.12 0)
+      (effects (font (size 1.27 1.27)))
+    )
+    (property "Footprint" "" (at 72.39 72.39 0)
+      (effects (font (size 1.27 1.27)) hide)
+    )
+    (property "Datasheet" "" (at 72.39 72.39 0)
       (effects (font (size 1.27 1.27)) hide)
     )
@@
         (path "/a45f22c9-49d1-4ac0-b785-e9b55c296b2a"
           (reference "SW1") (unit 1)
+        )
+      )
+    )
+  )
+  (symbol (lib_id "power:+5V") (at 72.39 78.74 0) (unit 1)
+    (in_bom yes) (on_board yes) (dnp no)
+    (property "Reference" "#PWR04" (at 72.39 82.55 0)
+      (effects (font (size 1.27 1.27)) hide)
+    )
+    (property "Value" "+5V" (at 72.39 81.28 0)
+      (effects (font (size 1.27 1.27)))
+    )
+    (property "Footprint" "" (at 72.39 78.74 0)
+      (effects (font (size 1.27 1.27)) hide)
+    )
+    (property "Datasheet" "" (at 72.39 78.74 0)
+      (effects (font (size 1.27 1.27)) hide)
+    )
+    (pin "1")
+    (instances
+      (project "neutrino_display"
+        (path "/a45f22c9-49d1-4ac0-b785-e9b55c296b2a"
+          (reference "#PWR04") (unit 1)
         )
       )
@@
         )
       )
-    )
-  )
-  (symbol (lib_id "power:GND") (at 80.01 73.66 0) (unit 1)
-    (in_bom yes) (on_board yes) (dnp no) (fields_autoplaced)
-    (property "Reference" "#PWR04" (at 80.01 80.01 0)
-      (effects (font (size 1.27 1.27)) hide)
-    )
-    (property "Value" "GND" (at 80.01 78.74 0)
-      (effects (font (size 1.27 1.27)))
-    )
-    (property "Footprint" "" (at 80.01 73.66 0)
-      (effects (font (size 1.27 1.27)) hide)
-    )
-    (property "Datasheet" "" (at 80.01 73.66 0)
-      (effects (font (size 1.27 1.27)) hide)
-    )
-    (pin "1")
-    (instances
-      (project "neutrino_display"
-        (path "/a45f22c9-49d1-4ac0-b785-e9b55c296b2a"
-          (reference "#PWR04") (unit 1)
-        )
-      )
